File: ADC_prevodnik/ADC_prevodnik.kicad_pcb (KiCad board)
At the start: 2 copper layers, 9 parts, among them J1 Conn_01x10_Pin, J2 Conn_01x04_Pin, J3 Conn_01x02_Pin

Commit message: 200426
Routing:
- net /ADDR: track 50.7 -> 27.8 mm
- net /VCC: track 14.9 -> 24.2 mm
- net /GPIO 21: track 27.8 -> 26.1 mm
Changed lines of the file:
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@@
 	)
 	(setup
+		(stackup
+			(layer "F.SilkS"
+				(type "Top Silk Screen")
+			)
+			(layer "F.Paste"
+				(type "Top Solder Paste")
+			)
+			(layer "F.Mask"
+				(type "Top Solder Mask")
+				(thickness 0.01)
+			)
+			(layer "F.Cu"
+				(type "copper")
+				(thickness 0.035)
+			)
+			(layer "dielectric 1"
+				(type "core")
+				(thickness 1.51)
+				(material "FR4")
+				(epsilon_r 4.5)
+				(loss_tangent 0.02)
+			)
+			(layer "B.Cu"
+				(type "copper")
+				(thickness 0.035)
+			)
+			(layer "B.Mask"
+				(type "Bottom Solder Mask")
+				(thickness 0.01)
+			)
+			(layer "B.Paste"
+				(type "Bottom Solder Paste")
+			)
+			(layer "B.SilkS"
+				(type "Bottom Silk Screen")
+			)
+			(copper_finish "None")
+			(dielectric_constraints no)
+		)
 		(pad_to_mask_clearance 0)
 		(allow_soldermask_bridges_in_footprints no)
@@
 	)
 	(segment
-		(start 154.71 87.25)
-		(end 149.96 82.5)
-		(width 1)
+		(start 164.25 92.38)
+		(end 159.12 87.25)
+		(width 0.4)
 		(layer "F.Cu")
 		(net 4)
 	)
 	(segment
-		(start 155.04 87.25)
+		(start 149.96 82.5)
 		(end 154.71 87.25)
-		(width 1)
+		(width 0.4)
 		(layer "F.Cu")
 		(net 4)
@@
 		(start 159.12 87.25)
 		(end 155.04 87.25)
-		(width 1)
-		(layer "B.Cu")
+		(width 0.4)
+		(layer "F.Cu")
 		(net 4)
 	)
 	(segment
-		(start 164.25 92.38)
-		(end 159.12 87.25)
-		(width 1)
-		(layer "B.Cu")
+		(start 154.71 87.25)
+		(end 155.04 87.25)
+		(width 0.4)
+		(layer "F.Cu")
 		(net 4)
 	)
 	(segment
-		(start 165.901 85.649)
-		(end 164.25 87.3)
-		(width 1)
+		(start 142.29 87.25)
+		(end 149.96 87.25)
+		(width 0.4)
 		(layer "F.Cu")
 		(net 6)
 	)
 	(segment
-		(start 150.657265 79.68)
-		(end 148.459 81.878265)
-		(width 1)
+		(start 164.25 79.68)
+		(end 165.601 81.031)
+		(width 0.4)
 		(layer "F.Cu")
 		(net 6)
 	)
 	(segment
-		(start 164.25 79.68)
-		(end 165.901 81.331)
-		(width 1)
-		(layer "F.Cu")
-		(net 6)
-	)
-	(segment
-		(start 164.25 79.68)
-		(end 150.657265 79.68)
-		(width 1)
-		(layer "F.Cu")
-		(net 6)
-	)
-	(segment
-		(start 165.901 81.331)
-		(end 165.901 85.649)
-		(width 1)
-		(layer "F.Cu")
-		(net 6)
-	)
-	(segment
-		(start 148.459 85.749)
-		(end 149.96 87.25)
-		(width 1)
+		(start 165.601 81.031)
+		(end 165.601 85.949)
+		(width 0.4)
 		(layer "F.Cu")
 		(net 6)
@@
 		(start 140.5 85.46)
 		(end 142.29 87.25)
-		(width 1)
+		(width 0.4)
 		(layer "F.Cu")
 		(net 6)
@@
 		(start 149.96 87.25)
 		(end 149.96 95.79)
-		(width 1)
-		(layer "F.Cu")
-		(net 6)
-	)
-	(segment
-		(start 148.459 81.878265)
-		(end 148.459 85.749)
-		(width 1)
-		(layer "F.Cu")
-		(net 6)
-	)
-	(segment
-		(start 142.29 87.25)
-		(end 149.96 87.25)
-		(width 1)
+		(width 0.4)
 		(layer "F.Cu")
 		(net 6)
@@
 		(start 149.96 95.79)
 		(end 149.75 96)
-		(width 1)
+		(width 0.4)
+		(layer "F.Cu")
+		(net 6)
+	)
+	(segment
+		(start 165.601 85.949)
+		(end 164.25 87.3)
+		(width 0.4)
 		(layer "F.Cu")
 		(net 6)
@@
 		(start 146.28 77.14)
 		(end 164.25 77.14)
-		(width 1)
+		(width 0.4)
 		(layer "F.Cu")
 		(net 7)
@@
 		(start 140.5 82.92)
 		(end 146.28 77.14)
-		(width 1)
+		(width 0.4)
 		(layer "F.Cu")
 		(net 7)
 	)
 	(segment
-		(start 148.25 80.25)
-		(end 162.28 80.25)
-		(width 1)
+		(start 160.421 86.049)
+		(end 164.25 82.22)
+		(width 0.4)
 		(layer "B.Cu")
 		(net 8)
 	)
 	(segment
-		(start 162.28 80.25)
-		(end 164.25 82.22)
-		(width 1)
+		(start 140.5 88)
+		(end 142.451 86.049)
+		(width 0.4)
 		(layer "B.Cu")
 		(net 8)
 	)
 	(segment
-		(start 140.5 88)
-		(end 148.25 80.25)
-		(width 1)
+		(start 142.451 86.049)
+		(end 160.421 86.049)
+		(width 0.4)
 		(layer "B.Cu")
 		(net 8)
 	)
 	(segment
-		(start 140.5 90.54)
-		(end 146.28 84.76)
-		(width 1)
+		(start 158.47 90.54)
+		(end 164.25 84.76)
+		(width 0.4)
 		(layer "B.Cu")
 		(net 9)
 	)
 	(segment
-		(start 146.28 84.76)
-		(end 164.25 84.76)
-		(width 1)
+		(start 140.5 90.54)
+		(end 158.47 90.54)
+		(width 0.4)
 		(layer "B.Cu")
 		(net 9)
 	)
 	(segment
-		(start 156.541 94.209)
+		(start 148.4 82.05)
+		(end 148.4 83.55)
+		(width 0.4)
+		(layer "F.Cu")
+		(net 10)
+	)
+	(segment
+		(start 155.04 82.5)
+		(end 153.59 81.05)
+		(width 0.4)
+		(layer "F.Cu")
+		(net 10)
+	)
+	(segment
+		(start 148.4 83.55)
+		(end 154.75 89.9)
+		(width 0.4)
+		(layer "F.Cu")
+		(net 10)
+	)
+	(segment
+		(start 154.75 89.9)
 		(end 154.75 96)
-		(width 1)
+		(width 0.4)
 		(layer "F.Cu")
 		(net 10)
 	)
 	(segment
-		(start 156.541 84.001)
-		(end 156.541 94.209)
-		(width 1)
+		(start 153.59 81.05)
+		(end 149.4 81.05)
+		(width 0.4)
 		(layer "F.Cu")
 		(net 10)
 	)
 	(segment
-		(start 155.04 82.5)
-		(end 156.541 84.001)
-		(width 1)
+		(start 149.4 81.05)
+		(end 148.4 82.05)
+		(width 0.4)
 		(layer "F.Cu")
 		(net 10)

Commit message: 210426
Parts:
- moved H1 6.90 mm to (138.4, 78.0)
- moved H2 6.90 mm to (138.4, 99.2)
- moved J2 4.22 mm to (144.7, 82.8)
- moved H3 3.51 mm to (169.0, 78.0)
- moved H4 3.50 mm to (169.0, 99.2)
- moved J1 2.07 mm to (162.6, 75.9)
- moved R2 1.11 mm to (150.0, 86.1)
- moved J3 0.84 mm to (149.9, 95.2)
Connections:
- net /ADDR renamed /GND
Routing:
- net /GPIO 21: track 26.1 -> 58.6 mm
- net /GND: track 27.8 -> 0.30 mm
- net /GPIO 22: track 26.1 -> 48.8 mm
- net /3,3V: track 26.1 -> 20.7 mm
- net /A0: track 18.4 -> 16.2 mm
- net /VCC: track 24.2 -> 25.1 mm
- added copper zone on B.Cu, net /GND
Other:
- board outline added: 38.6 x 30.4 mm
