File: ADC_prevodnik/ADC_prevodnik.kicad_sch (KiCad schematic)
At the start: 9 parts, among them J1 Conn_01x10_Pin, J2 Conn_01x04_Pin, J3 Conn_01x02_Pin

Commit message: 210426
Connections:
- net ADDR renamed GND
Changed lines of the file:
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@@
 		)
 	)
-	(label "ADDR"
+	(label "GND"
 		(at 186.69 88.9 0)
 		(effects

Commit message: 280426
Parts:
- R1: value 2k -> 3k
Changed lines of the file:
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@@
 			)
 		)
-		(property "Value" "2k"
+		(property "Value" "3k"
 			(at 158.75 106.6799 0)
 			(effects
