File: H-mustek/H-mustek.kicad_sch (KiCad schematic)
At the start: 22 parts, among them J1 Conn_01x02_Pin, J2 Conn_01x02_Pin, Q1 IRF3205, Q2 IRF3205, Q3 IRF3205, Q4 IRF3205, U1 IR2153, U2 IR2153

Commit message: 280426
Other:
- title: (none) -> AD/AC střídač
- moved on the sheet: J1, J2
Changed lines of the file:
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@@
 	(generator_version "9.0")
 	(paper "A4")
+	(title_block
+		(title "AD/AC střídač")
+		(date "20.2.2026")
+	)
 	(junction
 		(at 101.6 74.93)
@@
 	(wire
 		(pts
-			(xy 50.8 132.08) (xy 45.72 132.08)
+			(xy 220.98 63.5) (xy 215.9 63.5)
 		)
 		(stroke
@@
 	(wire
 		(pts
-			(xy 52.07 148.59) (xy 45.72 148.59)
+			(xy 222.25 80.01) (xy 215.9 80.01)
 		)
 		(stroke
@@
 	(wire
 		(pts
-			(xy 52.07 151.13) (xy 45.72 151.13)
+			(xy 222.25 82.55) (xy 215.9 82.55)
 		)
 		(stroke
@@
 	)
 	(label "VCC"
-		(at 50.8 132.08 0)
+		(at 220.98 63.5 0)
 		(effects
 			(font
@@
 	)
 	(label "VOUT1"
-		(at 52.07 148.59 0)
+		(at 222.25 80.01 0)
 		(effects
 			(font
@@
 	)
 	(label "VOUT2"
-		(at 52.07 151.13 0)
+		(at 222.25 82.55 0)
 		(effects
 			(font
@@
 	(symbol
 		(lib_id "power:GND")
-		(at 45.72 134.62 0)
+		(at 215.9 66.04 0)
 		(unit 1)
 		(exclude_from_sim no)
@@
 		(fields_autoplaced yes)
 		(property "Reference" "#PWR03"
-			(at 45.72 140.97 0)
+			(at 215.9 72.39 0)
 			(effects
 				(font
@@
 		)
 		(property "Value" "GND"
-			(at 45.72 139.7 0)
+			(at 215.9 71.12 0)
 			(effects
 				(font
@@
 		)
 		(property "Footprint" ""
-			(at 45.72 134.62 0)
+			(at 215.9 66.04 0)
 			(effects
 				(font
@@
 		)
 		(property "Datasheet" ""
-			(at 45.72 134.62 0)
+			(at 215.9 66.04 0)
 			(effects
 				(font
@@
 		)
 		(property "Description" "Power symbol creates a global label with name \"GND\" , ground"
-			(at 45.72 134.62 0)
+			(at 215.9 66.04 0)
 			(effects
 				(font
@@
 	(symbol
 		(lib_id "Connector:Conn_01x02_Pin")
-		(at 40.64 148.59 0)
+		(at 210.82 80.01 0)
 		(unit 1)
 		(exclude_from_sim no)
@@
 		(fields_autoplaced yes)
 		(property "Reference" "J2"
-			(at 41.275 143.51 0)
+			(at 211.455 74.93 0)
 			(effects
 				(font
@@
 		)
 		(property "Value" "Conn_01x02_Pin"
-			(at 41.275 146.05 0)
+			(at 211.455 77.47 0)
 			(effects
 				(font
@@
 		)
 		(property "Footprint" "Connector_Wire:SolderWire-2.5sqmm_1x02_P7.2mm_D2.4mm_OD3.6mm"
-			(at 40.64 148.59 0)
+			(at 210.82 80.01 0)
 			(effects
 				(font
@@
 		)
 		(property "Datasheet" "~"
-			(at 40.64 148.59 0)
+			(at 210.82 80.01 0)
 			(effects
 				(font
@@
 		)
 		(property "Description" "Generic connector, single row, 01x02, script generated"
-			(at 40.64 148.59 0)
+			(at 210.82 80.01 0)
 			(effects
 				(font
@@
 	(symbol
 		(lib_id "Connector:Conn_01x02_Pin")
-		(at 40.64 132.08 0)
+		(at 210.82 63.5 0)
 		(unit 1)
 		(exclude_from_sim no)
@@
 		(fields_autoplaced yes)
 		(property "Reference" "J1"
-			(at 41.275 127 0)
+			(at 211.455 58.42 0)
 			(effects
 				(font
@@
 		)
 		(property "Value" "Conn_01x02_Pin"
-			(at 41.275 129.54 0)
+			(at 211.455 60.96 0)
 			(effects
 				(font
@@
 		)
 		(property "Footprint" "Connector_AMASS:AMASS_XT30UPB-F_1x02_P5.0mm_Vertical"
-			(at 40.64 132.08 0)
+			(at 210.82 63.5 0)
 			(effects
 				(font
@@
 		)
 		(property "Datasheet" "~"
-			(at 40.64 132.08 0)
+			(at 210.82 63.5 0)
 			(effects
 				(font
@@
 		)
 		(property "Description" "Generic connector, single row, 01x02, script generated"
-			(at 40.64 132.08 0)
-			(effects
-				(font
+			(at 210.82 63.5 0)
+			(effects
+				(font
