File: usmernovac/usmernovac.kicad_pcb (KiCad board)
At the start: 2 copper layers, 11 parts, among them J1 Conn_01x02_Pin, J2 Conn_01x02_Pin

Commit message: 260426
Routing:
- net GND: track 48.8 -> 0.00 mm
- net /VOUT: track 47.6 -> 36.2 mm
- added copper zone on B.Cu, net GND
Other:
- board outline added: 60 x 35 mm
Changed lines of the file:
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@@
 	)
 	(gr_rect
-		(start 122.5 60)
-		(end 182.5 95)
+		(start 122.55 60)
+		(end 182.5 94.95)
 		(stroke
-			(width 0.2)
+			(width 0.05)
 			(type default)
 		)
 		(fill no)
-		(layer "F.Cu")
+		(layer "Edge.Cuts")
+	)
+	(segment
+		(start 152.5 75)
+		(end 152.5 70.08)
+		(width 0.8)
+		(layer "B.Cu")
+		(net 1)
+	)
+	(segment
+		(start 152.5 70.08)
+		(end 157.58 65)
+		(width 0.8)
+		(layer "B.Cu")
+		(net 1)
 	)
 	(segment
 		(start 157.58 65)
-		(end 157.58 69.92)
+		(end 165 72.42)
 		(width 0.8)
-		(layer "F.Cu")
+		(layer "B.Cu")
 		(net 1)
 	)
 	(segment
-		(start 165 72.42)
-		(end 157.58 65)
+		(start 167.58 75)
+		(end 165 72.42)
 		(width 0.8)
-		(layer "F.Cu")
+		(layer "B.Cu")
 		(net 1)
 	)
 	(segment
-		(start 152.5 75)
-		(end 177.5 75)
+		(start 177.5 75)
+		(end 167.58 75)
 		(width 0.8)
-		(layer "F.Cu")
+		(layer "B.Cu")
 		(net 1)
 	)
 	(segment
-		(start 157.58 69.92)
-		(end 152.5 75)
+		(start 127.5 75)
+		(end 137.42 75)
 		(width 0.8)
-		(layer "F.Cu")
-		(net 1)
-	)
-	(segment
-		(start 132.58 72.42)
-		(end 140 72.42)
-		(width 0.8)
-		(layer "F.Cu")
+		(layer "B.Cu")
 		(net 2)
 	)
 	(segment
-		(start 127.5 75)
-		(end 130 75)
+		(start 137.42 75)
+		(end 140 72.42)
 		(width 0.8)
-		(layer "F.Cu")
+		(layer "B.Cu")
 		(net 2)
 	)
 	(segment
-		(start 130 75)
-		(end 132.58 72.42)
+		(start 140 72.42)
+		(end 147.42 65)
 		(width 0.8)
-		(layer "F.Cu")
+		(layer "B.Cu")
 		(net 2)
 	)
 	(segment
-		(start 147.42 65)
-		(end 140 72.42)
+		(start 127.5 82.8)
+		(end 136.701 92.001)
 		(width 0.8)
-		(layer "F.Cu")
-		(net 2)
-	)
-	(segment
-		(start 147.42 85.08)
-		(end 152.5 80)
-		(width 0.8)
-		(layer "F.Cu")
-		(net 3)
-	)
-	(segment
-		(start 147.42 90)
-		(end 147.42 85.08)
-		(width 0.8)
-		(layer "F.Cu")
-		(net 3)
-	)
-	(segment
-		(start 140 82.58)
-		(end 147.42 90)
-		(width 0.8)
-		(layer "F.Cu")
-		(net 3)
-	)
-	(segment
-		(start 152.5 80)
-		(end 174.7 80)
-		(width 0.8)
-		(layer "F.Cu")
-		(net 3)
-	)
-	(segment
-		(start 174.7 80)
-		(end 177.5 82.8)
-		(width 0.8)
-		(layer "F.Cu")
-		(net 3)
-	)
-	(segment
-		(start 127.5 82.8)
-		(end 137.2 92.5)
-		(width 0.8)
-		(layer "F.Cu")
+		(layer "B.Cu")
 		(net 4)
 	)
 	(segment
-		(start 155.08 92.5)
-		(end 157.58 90)
+		(start 157.58 90)
+		(end 165 82.58)
 		(width 0.8)
-		(layer "F.Cu")
+		(layer "B.Cu")
 		(net 4)
 	)
 	(segment
-		(start 137.2 92.5)
-		(end 155.08 92.5)
+		(start 136.701 92.001)
+		(end 155.579 92.001)
 		(width 0.8)
-		(layer "F.Cu")
+		(layer "B.Cu")
 		(net 4)
 	)
 	(segment
-		(start 165 82.58)
+		(start 155.579 92.001)
 		(end 157.58 90)
 		(width 0.8)
-		(layer "F.Cu")
+		(layer "B.Cu")
 		(net 4)
 	)
+	(zone
+		(net 3)
+		(net_name "GND")
+		(layer "B.Cu")
+		(hatch edge 0.5)
+		(connect_pads
+			(clearance 0.5)
+		)
+		(min_thickness 0.25)
+		(filled_areas_thickness no)
+		(fill yes
+			(thermal_gap 0.5)
+			(thermal_bridge_width 0.5)
+		)
+		(polygon
+			(pts
+				(xy 122.55 94.95) (xy 182.5 94.95) (xy 182.5 60) (xy 122.55 60) (xy 122.55 94.95)
+			)
+		)
+	)
 	(embedded_fonts no)
