File: usmernovac/usmernovac.kicad_sch (KiCad schematic)
At the start: 11 parts, among them J1 Conn_01x02_Pin, J2 Conn_01x02_Pin

Commit message: 280426
Other:
- title: (none) -> Usměrňovač
- moved on the sheet: C1, D1, D2, D3, D4, H1, H2, H3, H4, J1, J2
